Commit message: setting up franka panda simulation

File: panda_example/assets/franka_panda/panda.urdf (robot description, URDF)
Before this commit: robot panda, 13 links, 12 joints
Links:
- removed link panda_grasptarget
- removed link panda_leftfinger
- removed link panda_rightfinger
- added link panda_centerfinger, mass 0.1; collision mesh filename=package://meshes/collision/cylinder.obj; visual mesh filename=package://meshes/visual/cylinder.obj
Joints:
- removed joint panda_finger_joint1
- removed joint panda_finger_joint2
- removed joint panda_grasptarget_hand
- added joint panda_centerfinger_joint: type prismatic, parent panda_hand, child panda_centerfinger, origin xyz=0 0 0.0584 rpy=0 0 0, axis 0 0 1, limit lower=0.0 upper=0.04 effort=20 velocity=0.2
